Commit message: Update backpack_3d.urdf

File: cartographer_ros/urdf/backpack_3d.urdf (robot description, URDF)
Before this commit: robot cartographer_backpack_3d, 4 links, 3 joints
Links:
- removed link horizontal_vlp16_link
- removed link vertical_vlp16_link
- added link velodyne; visual cylinder length=0.07 radius=0.05
Joints:
- removed joint horizontal_vlp16_link_joint
- removed joint vertical_vlp16_link_joint
- added joint velodyne_joint: type fixed, parent base_link, child velodyne, origin xyz=0 0 0 rpy=0 0 0
- joint imu_link_joint: origin xyz=0 0 0 rpy=3.1416 0 0 -> xyz=0 0 0 rpy=0 0 0

Commit message: Update backpack_3d.urdf

File: cartographer_ros/urdf/backpack_3d.urdf (robot description, URDF)
Before this commit: robot stencil, 3 links, 2 joints
Links:
- removed link velodyne
- added link vertical_vlp16_link; visual cylinder length=0.07 radius=0.05
Joints:
- removed joint velodyne_joint
- added joint vertical_vlp16_link_joint: type fixed, parent base_link, child vertical_vlp16_link, origin xyz=0.0 0.0 0.0 rpy=3.14 0.0 0.0
